Commit message: camrea urdf, launch_robot added

File: description/lidar.xacro (robot description, xacro)
@@ -4,10 +4,10 @@
         <parent link="chassis"/>
         <child link="laser_frame"/>
-        <origin xyz="0.33 0 0.145" rpy="0 0 0"/>
+        <origin xyz="0.33 0 0.170" rpy="0 0 0"/>
     </joint>
     <link name="laser_frame">
         <visual>
             <geometry>
-                <cylinder radius="0.05" length="0.04"/>
+                <cylinder radius="0.05" length="0.040"/>
             </geometry>
             <material name="red"/>

File: description/robot.urdf.xacro (robot description, xacro)
@@ -4,3 +4,4 @@
     <xacro:include filename="lidar.xacro" />
     <xacro:include filename="ros2_control.xacro" />
+    <xacro:include filename="camera.xacro" />
 </robot>

File: description/robot_core.xacro (robot description, xacro)
@@ -22,4 +22,7 @@
         <color rgba="1 0 0 1"/>
     </material>
+    <material name="greyishteal" >
+        <color rgba="0.44313725490196076 0.6235294117647059 0.5686274509803921 1.0" />
+    </material>
     <link name="base_link">
     </link>
@@ -33,5 +36,12 @@
             <origin xyz="0.17 0 0.06" rpy="0 0 0"/>
             <geometry>
-               <box size="0.34 0.30 0.12"/>
+               <box size="0.34 0.30 0.02"/>
+            </geometry>
+            <material name="grey"/>
+        </visual>
+        <visual>
+            <origin xyz="0.330 0 0.10" rpy="0 0 0"/>
+            <geometry>
+               <box size="0.020 0.020 0.100"/>
             </geometry>
             <material name="grey"/>

Commit message: new chasis dimentions

File: description/lidar.xacro (robot description, xacro)
@@ -4,10 +4,10 @@
         <parent link="chassis"/>
         <child link="laser_frame"/>
-        <origin xyz="0.33 0 0.170" rpy="0 0 0"/>
+        <origin xyz="0.220 0 0.111" rpy="0 0 0"/>
     </joint>
     <link name="laser_frame">
         <visual>
             <geometry>
-                <cylinder radius="0.05" length="0.040"/>
+                <cylinder radius="0.050" length="0.040"/>
             </geometry>
             <material name="red"/>

File: description/robot_core.xacro (robot description, xacro)
@@ -30,15 +30,15 @@
         <parent link="base_link"/>
         <child link="chassis"/>
-        <origin xyz="-0.1 0 0"/>
+        <origin xyz="-0.090 0 0"/>
     </joint>
     <link name="chassis">
         <visual>
-            <origin xyz="0.17 0 0.06" rpy="0 0 0"/>
+            <origin xyz="0.145 0 0.0455" rpy="0 0 0"/>
             <geometry>
-               <box size="0.34 0.30 0.02"/>
+               <box size="0.290 0.190 0.091"/>
             </geometry>
             <material name="grey"/>
         </visual>
-        <visual>
+        <!--<visual>
             <origin xyz="0.330 0 0.10" rpy="0 0 0"/>
             <geometry>
@@ -46,5 +46,5 @@
             </geometry>
             <material name="grey"/>
-        </visual>
+        </visual>-->
     </link>
         <!-- LEFT WHEEL -->
@@ -52,5 +52,5 @@
         <parent link="base_link"/>
         <child link="left_wheel"/>
-        <origin xyz="0 0.172 0" rpy="-${pi/2} 0 0"/>
+        <origin xyz="0 0.102 0" rpy="-${pi/2} 0 0"/>
         <axis xyz="0 0 1"/>
     </joint>
@@ -67,5 +67,5 @@
         <parent link="base_link"/>
         <child link="right_wheel"/>
-        <origin xyz="0 -0.172 0" rpy="${pi/2} 0 0"/>
+        <origin xyz="0 -0.102 0" rpy="${pi/2} 0 0"/>
         <axis xyz="0 0 -1"/>
     </joint>
@@ -82,5 +82,5 @@
         <parent link="chassis"/>
         <child link="caster_wheel"/>
-        <origin xyz="0.33 0 0" rpy="0 0 0"/>
+        <origin xyz="0.280 0 0" rpy="0 0 0"/>
     </joint>
     <link name="caster_wheel">
