Commit message: lidar urdf added

File: description/robot_core.xacro (robot description, xacro)
@@ -18,4 +18,7 @@
     <material name="lightgrey" >
         <color rgba="0.8470588235294118 0.8627450980392157 0.8392156862745098 1.0" />
+    </material>
+    <material name="red">
+        <color rgba="1 0 0 1"/>
     </material>
     <link name="base_link">
@@ -45,5 +48,5 @@
         <visual>
             <geometry>
-                <cylinder length="0.034" radius="0.060" />
+                <cylinder length="0.033" radius="0.060" />
             </geometry>
             <material name="black"/>
@@ -69,5 +72,5 @@
         <parent link="chassis"/>
         <child link="caster_wheel"/>
-        <origin xyz="0.34 0 0" rpy="0 0 0"/>
+        <origin xyz="0.33 0 0" rpy="0 0 0"/>
     </joint>
     <link name="caster_wheel">

Commit message: urdf right wheeljoint rpy changed

File: description/robot_core.xacro (robot description, xacro)
@@ -67,5 +67,5 @@
         <parent link="base_link"/>
         <child link="right_wheel"/>
-        <origin xyz="0 -0.102 0" rpy="${pi/2} 0 0"/>
+        <origin xyz="0 -0.102 0" rpy="-${pi/2} 0 ${pi}"/>
         <axis xyz="0 0 -1"/>
     </joint>
